File: KiCad/Register_File/GP_Register/Register_1.0.kicad_sch (KiCad schematic)
At the start: 59 parts, among them J1 Conn_01x02_Pin, J2 Conn_01x02_Pin, J3 Conn_01x02_Pin, J4 Conn_01x08_Pin, J5 Conn_01x08_Pin, J6 Conn_01x04_Pin, J7 Conn_01x04_Pin, J8 Conn_01x04_Pin, J9 Conn_01x04_Pin, SW1 SW_SPDT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

Commit message: finished registier file boards
Changed lines of the file:
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@@
 		)
 	)
-	(label "B[0..15]"
+	(label "Y[0..15]"
 		(at 339.09 50.8 0)
 		(fields_autoplaced yes)
