File: KiCad/Program_Counter/Program_Counter.kicad_sch (KiCad schematic)
At the start: 28 parts, among them J1 Conn_01x08_Socket, J2 Conn_01x08_Socket, J3 Conn_01x05_Socket, J4 Conn_01x02_Socket, U1 74LS161, U2 74LS161, U3 74LS161, U4 74LS161, U5 74LS245, U6 74LS245

Commit message: finished registier file boards
Parts:
- removed J2: Conn_01x08_Socket, Connector_JST:JST_XH_S8B-XH-A_1x08_P2.50mm_Horizontal, symbol Connector:Conn_01x08_Socket
- removed J3: Conn_01x05_Socket, Connector_JST:JST_XH_S5B-XH-A_1x05_P2.50mm_Horizontal, symbol Connector:Conn_01x05_Socket
- added H1, H2, H3, H4: MountingHole_Pad, MountingHole:MountingHole_2.2mm_M2_DIN965_Pad, symbol Mechanical:MountingHole_Pad
- added J3: Conn_01x08_Socket, Connector_JST:JST_XH_S8B-XH-A_1x08_P2.50mm_Horizontal, symbol Connector:Conn_01x08_Socket
- added J5: Conn_01x02_Socket, Connector_JST:JST_XH_S2B-XH-A_1x02_P2.50mm_Horizontal, symbol Connector:Conn_01x02_Socket
- added J6: Conn_01x03_Socket, Connector_JST:JST_XH_S3B-XH-A-1_1x03_P2.50mm_Horizontal, symbol Connector:Conn_01x03_Socket
- D0, D1, D10, D11, D12, D13, D14, D15, D2, D3, D4, D5, D6, D7, D8, D9: footprint LED_THT:LED_Rectangular_W5.0mm_H2.0mm_Horizontal_O1.27mm_Z3.0mm -> LED_THT:LED_Rectangular_W3.0mm_H2.0mm
Connections:
- net CLK: now also J5.2 (Pin_2)
- net D0: now also J3.1 (Pin_1); no longer J1.8 (Pin_8)
- net D1: now also J3.2 (Pin_2); no longer J1.7 (Pin_7)
- net D10: now also J1.3 (Pin_3)
- net D11: now also J1.4 (Pin_4)
- net D12: now also J1.5 (Pin_5)
- net D13: now also J1.6 (Pin_6)
- net D14: now also J1.7 (Pin_7)
- net D15: now also J1.8 (Pin_8)
- net D2: now also J3.3 (Pin_3); no longer J1.6 (Pin_6)
- net D3: now also J3.4 (Pin_4); no longer J1.5 (Pin_5)
- net D4: now also J3.5 (Pin_5); no longer J1.4 (Pin_4)
- net D5: now also J3.6 (Pin_6); no longer J1.3 (Pin_3)
- net D6: now also J3.7 (Pin_7); no longer J1.2 (Pin_2)
- net D7: now also J3.8 (Pin_8); no longer J1.1 (Pin_1)
- net D8: now also J1.1 (Pin_1)
- net D9: now also J1.2 (Pin_2)
- net GND: now also H1.1, H2.1, H3.1, H4.1
- net MR: now also J5.1 (Pin_1)
- net PC_INC: now also J6.2 (Pin_2)
- net PC_LOAD: now also J6.1 (Pin_1)
- net PC_OUT: now also J6.3 (Pin_3)
Other:
- note added: "Connectors"
- note added: "Mounting holes"
- moved on the sheet: J4

Commit message: added con_ctrl board mdr_mar
Parts:
- removed J5: Conn_01x02_Socket, Connector_JST:JST_XH_S2B-XH-A_1x02_P2.50mm_Horizontal, symbol Connector:Conn_01x02_Socket
- added J2: Conn_01x02_Socket, Connector_JST:JST_XH_S2B-XH-A_1x02_P2.50mm_Horizontal, symbol Connector:Conn_01x02_Socket
Connections:
- net CLK: now also J2.1 (Pin_1)
- net MR: now also J2.2 (Pin_2)
Changed lines of the file:
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@@
+	)
+	(symbol
+		(lib_id "Connector:Conn_01x02_Socket")
+		(at 26.67 96.52 0)
+		(mirror y)
+		(unit 1)
+		(exclude_from_sim no)
+		(in_bom yes)
+		(on_board yes)
+		(dnp no)
+		(property "Reference" "J2"
+			(at 26.67 94.488 0)
+			(effects
+				(font
+					(size 1.27 1.27)
+				)
+			)
+		)
+		(property "Value" "Conn_01x02_Socket"
+			(at 27.305 101.6 0)
+			(effects
+				(font
+					(size 1.27 1.27)
+				)
+				(hide yes)
+			)
+		)
+		(property "Footprint" "Connector_JST:JST_XH_S2B-XH-A_1x02_P2.50mm_Horizontal"
+			(at 26.67 96.52 0)
+			(effects
+				(font
+					(size 1.27 1.27)
+				)
+				(hide yes)
+			)
+		)
+		(property "Datasheet" "~"
+			(at 26.67 96.52 0)
+			(effects
+				(font
+					(size 1.27 1.27)
+				)
+				(hide yes)
+			)
+		)
+		(property "Description" "Generic connector, single row, 01x02, script generated"
+			(at 26.67 96.52 0)
+			(effects
+				(font
+					(size 1.27 1.27)
+				)
+				(hide yes)
+			)
+		)
+		(pin "2"
+		)
+		(pin "1"
+		)
+		(instances
+			(project "Program_Counter"
+				(path "/2a73fea7-d07b-4c99-8a39-1d8877febd0a"
+					(reference "J2")
+					(unit 1)
+				)
+			)
+		)
 	)
 	(symbol
@@
 					(unit 1)
 				)
-			)
-		)
-	)
-	(symbol
-		(lib_id "Connector:Conn_01x02_Socket")
-		(at 26.67 99.06 180)
-		(unit 1)
-		(exclude_from_sim no)
-		(in_bom yes)
-		(on_board yes)
-		(dnp no)
-		(property "Reference" "J5"
-			(at 27.305 94.615 0)
-			(effects
-				(font
-					(size 1.27 1.27)
-				)
-			)
-		)
-		(property "Value" "Conn_01x02_Socket"
-			(at 27.305 93.98 0)
-			(effects
-				(font
-					(size 1.27 1.27)
-				)
-				(hide yes)
-			)
-		)
-		(property "Footprint" "Connector_JST:JST_XH_S2B-XH-A_1x02_P2.50mm_Horizontal"
-			(at 26.67 99.06 0)
-			(effects
-				(font
-					(size 1.27 1.27)
-				)
-				(hide yes)
-			)
-		)
-		(property "Datasheet" "~"
-			(at 26.67 99.06 0)
-			(effects
-				(font
-					(size 1.27 1.27)
-				)
-				(hide yes)
-			)
-		)
-		(property "Description" "Generic connector, single row, 01x02, script generated"
-			(at 26.67 99.06 0)
-			(effects
-				(font
-					(size 1.27 1.27)
-				)
-				(hide yes)
-			)
-		)
-		(pin "2"
-		)
-		(pin "1"
-		)
-		(instances
-			(project "Program_Counter"
-				(path "/2a73fea7-d07b-4c99-8a39-1d8877febd0a"
-					(reference "J5")
-					(unit 1)
-				)
