File: KiCad/Instruction_Register/Instruction_Register.kicad_pcb (KiCad board)
At the start: 2 copper layers, 100 x 100 mm, 55 parts, among them J1 Conn_01x02_Pin, J2 Conn_01x02_Pin, J3 Conn_01x02_Pin, J4 Conn_01x08_Pin, J5 Conn_01x08_Pin, J6 Conn_01x05_Pin, J7 Conn_01x02_Pin, J8 Conn_01x04_Pin, J9 Conn_01x04_Pin, SW1 SW_SPDT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

Commit message: added con_ctrl board mdr_mar
Parts:
- R1, R10, R12, R13, R14, R15, R16, R2, R3, R4, R5, R6, R7, R8, R9: footprint Resistor_THT:R_Axial_DIN0204_L3.6mm_D1.6mm_P7.62mm_Horizontal -> Resistor_SMD:R_1206_3216Metric
- moved R10 6.09 mm to (140.8, 58.4)
- moved R9 6.09 mm to (137.0, 58.4)
- moved R12 6.05 mm to (155.5, 58.5)
- moved R13 6.05 mm to (159.2, 58.5)
- moved R14 6.05 mm to (162.9, 58.5)
- moved R15 6.05 mm to (166.6, 58.5)
- moved R16 6.05 mm to (170.2, 58.5)
- moved R1 6.00 mm to (108.8, 107.8)
- moved R2 6.00 mm to (108.8, 104.0)
- moved R3 6.00 mm to (108.8, 100.2)
- moved R4 6.00 mm to (108.8, 96.5)
- moved R5 5.95 mm to (108.9, 73.0)
- moved R6 5.95 mm to (108.9, 69.2)
- moved R7 5.95 mm to (108.9, 65.2)
- moved R8 5.91 mm to (108.9, 61.5)
Routing:
- net /Y7: track 72.1 -> 79.7 mm
- net /Y5: track 57.1 -> 64.1 mm
- net /Y4: track 51.1 -> 57.5 mm, vias 0 -> 1
- net /V_OUT: track 27.0 -> 33.4 mm
- net /Y6: track 64.8 -> 70.8 mm, vias 1 -> 2
- net /Y3: track 71.2 -> 76.1 mm
- net /Y12: track 57.9 -> 62.5 mm
- net /Y14: track 52.6 -> 57.2 mm
- net /Y13: track 54.9 -> 59.5 mm
- net /Y8: track 57.3 -> 61.6 mm
- net /RST: track 131.6 -> 135.7 mm, vias 1 -> 2
- net /Y15: track 49.8 -> 53.2 mm, vias 0 -> 1
- net /IR_IN: track 154.0 -> 156.9 mm, vias 1 -> 0
- net /Y11: track 80.2 -> 78.0 mm, vias 0 -> 1
- net Net-(D8-A): track 2.19 -> 0.00 mm
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