File: KiCad/ALU/ALU_Main/ALU_Main.kicad_pcb (KiCad board)
At the start: 2 copper layers, 100 x 100 mm, 46 parts, among them J1 Conn_01x02_Socket, J2 Conn_01x04_Socket, J3 Conn_01x05_Socket, J4 Conn_01x16_Socket, J5 Conn_01x16_Socket, J8 Conn_01x16_Socket, U1 74LS181, U2 74LS181, U3 74LS181, U4 74LS181

Commit message: .
Parts:
- removed D0, D1, D10, D11, D12, D13, D14, D15, D2, D3, D4, D5, D6, D7, D8, D9: LED, LED_SMD:LED_1206_3216Metric_Pad1.42x1.75mm_HandSolder
- removed R0, R1, R10, R11, R12, R13, R14, R15, R2, R3, R4, R5, R6, R7, R8, R9: R_US, Resistor_SMD:R_1206_3216Metric_Pad1.30x1.75mm_HandSolder
- added J10: Conn_01x08_Socket, Connector_JST:JST_XH_S8B-XH-A-1_1x08_P2.50mm_Horizontal, F.Cu at (108.0, 116.0)
- added J6: Conn_01x08_Socket, Connector_JST:JST_XH_S8B-XH-A-1_1x08_P2.50mm_Horizontal, F.Cu at (163.5, 58.0)
- added J7: Conn_01x08_Socket, Connector_JST:JST_XH_S8B-XH-A-1_1x08_P2.50mm_Horizontal, F.Cu at (192.0, 133.5)
- added J9: Conn_01x08_Socket, Connector_JST:JST_XH_S8B-XH-A-1_1x08_P2.50mm_Horizontal, F.Cu at (108.0, 91.5)
- J4: value Conn_01x16_Socket -> Conn_01x02_Socket; footprint Connector_IDC:IDC-Header_2x08_P2.54mm_Horizontal -> Connector_JST:JST_XH_S2B-XH-A-1_1x02_P2.50mm_Horizontal
- J5, J8: value Conn_01x16_Socket -> Conn_01x08_Socket; footprint Connector_IDC:IDC-Header_2x08_P2.54mm_Horizontal -> Connector_JST:JST_XH_S8B-XH-A-1_1x08_P2.50mm_Horizontal
- moved J4 101.7 mm to (121.5, 142.0)
- moved J5 52.2 mm to (188.0, 58.0)
- moved J8 46.1 mm to (192.0, 109.0)
- moved J2 43.9 mm to (148.0, 142.0)
- moved J1 36.5 mm to (112.0, 142.0)
- moved U2 30.1 mm to (159.6, 69.8), turned to 0 degrees
- moved H1 30.0 mm to (104.0, 54.0)
- moved H2 30.0 mm to (196.0, 54.0)
- moved H3 30.0 mm to (104.0, 146.0)
- moved H4 30.0 mm to (196.0, 146.0)
- moved J3 29.6 mm to (131.0, 142.0)
- moved U1 28.3 mm to (124.4, 70.4), turned to 0 degrees
- moved U4 24.8 mm to (159.2, 104.5), turned to 0 degrees
- moved U3 24.1 mm to (124.2, 104.1), turned to 0 degrees
Connections:
- J2 pad 1: unconnected-(J2-Pin_1-Pad1) -> ~{C_{in}}
- J2 pad 2: unconnected-(J2-Pin_2-Pad2) -> ~{C_{out}}
- J4 pad 1: A_0 -> VCC
- J4 pad 2: A_1 -> GND
- J5 pad 1: B_0 -> F_0
- J5 pad 2: B_1 -> F_1
- J5 pad 3: B_2 -> F_2
- J5 pad 4: B_3 -> F_3
- J5 pad 5: B_4 -> F_4
- J5 pad 6: B_5 -> F_5
- J5 pad 7: B_6 -> F_6
- J5 pad 8: B_7 -> F_7
- J8 pad 1: F_0 -> A_8
- J8 pad 2: F_1 -> A_9
- J8 pad 3: F_2 -> A_10
- J8 pad 4: F_3 -> A_11
- J8 pad 5: F_4 -> A_12
- J8 pad 6: F_5 -> A_13
- J8 pad 7: F_6 -> A_14
- J8 pad 8: F_7 -> A_15
Routing:
- net VCC: track 0.00 -> 14.1 mm
